Commit message: control plant framework complete

File: workspace/centuar_sim/centaur_v3.urdf (robot description, URDF)
Before this commit: robot centuar, 11 links, 10 joints
Joints:
- joint left_foot_fixed_joint: origin xyz=0 0 -0.445 rpy=0 0 0 -> xyz=0 0 -0.455 rpy=0 0 0
- joint right_foot_fixed_joint: origin xyz=0 0 -0.445 rpy=0 0 0 -> xyz=0 0 -0.455 rpy=0 0 0
